Commit message: update inertia

File: urdf/hopejr_hand.urdf (robot description, URDF)
Before this commit: robot hopejr_hand, 46 links, 45 joints
Links:
- link base_link: mass 2.0 -> 0.03323
- link hand: mass 2.0 -> 0.252893
- link index_dip_1: mass 2.0 -> 0.005093
- link index_dip_2: mass 2.0 -> 0.005429
- link index_mcp_1: mass 2.0 -> 0.004836
- link index_mcp_2: mass 2.0 -> 0.001654
- link index_pip: mass 2.0 -> 0.005708
- link middle_dip_1: mass 2.0 -> 0.005093
- link middle_dip_2: mass 2.0 -> 0.005429
- link middle_mcp_1: mass 2.0 -> 0.004836
- link middle_mcp_2: mass 2.0 -> 0.001654
- link middle_pip: mass 2.0 -> 0.005708
- link pinky_dip_1: mass 2.0 -> 0.005093
- link pinky_dip_2: mass 2.0 -> 0.005429
- link pinky_mcp_1: mass 2.0 -> 0.004836
- link pinky_mcp_2: mass 2.0 -> 0.001654
- link pinky_pip: mass 2.0 -> 0.005708
- link ring_dip_1: mass 2.0 -> 0.005093
- link ring_dip_2: mass 2.0 -> 0.005429
- link ring_mcp_1: mass 2.0 -> 0.004836
- link ring_mcp_2: mass 2.0 -> 0.001654
- link ring_pip: mass 2.0 -> 0.005708
- link thumb_dip: mass 2.0 -> 0.005429
- link thumb_mcp_2: mass 2.0 -> 0.008776
- link thumb_pip_1: mass 2.0 -> 0.007142
- link thumb_pip_2: mass 2.0 -> 0.006089

File: urdf/hopejr_hand.urdf.xacro (robot description, xacro)
@@ -18,6 +18,6 @@
             <inertial>
                 <origin xyz="-0.02 0 0.028" rpy="0 0 0"/>
-                <mass value="2.0"/>
-                <inertia ixx="0.000213" ixy="0" ixz="0" iyy="0.007034" iyz="0" izz="0.008104"/>
+                <mass value="0.03323"/>
+                <inertia ixx="0.000018824494" ixy="-0.000000571474" ixz="-0.000000041098" iyy="0.00001505929" iyz="0.000000023636" izz="0.000013661405"/>
             </inertial>
         </link>
@@ -37,6 +37,6 @@
             <inertial>
                 <origin xyz="0 0 0" rpy="0 0 0"/>
-                <mass value="2.0"/>
-                <inertia ixx="0.01" ixy="0" ixz="0" iyy="0.01" iyz="0" izz="0.01"/>
+                <mass value="0.252893"/>
+                <inertia ixx="0.0002839" ixy="0.000003336317" ixz="0.000004077546" iyy="0.0001891" iyz="0.000000331897" izz="0.0001469"/>
             </inertial>
         </link>
@@ -63,6 +63,6 @@
             <inertial>
                 <origin xyz="0 0 0" rpy="0 0 0"/>
-                <mass value="2.0"/>
-                <inertia ixx="0.001" ixy="0" ixz="0" iyy="0.001" iyz="0" izz="0.001"/>
+                <mass value="0.008776"/>
+                <inertia ixx="0.000000783215" ixy="0.000000007992" ixz="0.000000266897" iyy="0.000000932685" iyz="-0.000000055174" izz="0.000000534905"/>
             </inertial>
         </link>
@@ -103,6 +103,6 @@
             <inertial>
                 <origin xyz="0 0 0" rpy="0 0 0"/>
-                <mass value="2.0"/>
-                <inertia ixx="0.001" ixy="0" ixz="0" iyy="0.001" iyz="0" izz="0.001"/>
+                <mass value="0.007142"/>
+                <inertia ixx="0.000000233324" ixy="-0.000000000007" ixz="0.00000000023" iyy="0.000000597862" iyz="0.000000000054" izz="0.000000638412"/>
             </inertial>
         </link>
@@ -143,6 +143,6 @@
             <inertial>
                 <origin xyz="0 0 0" rpy="0 0 0"/>
-                <mass value="2.0"/>
-                <inertia ixx="0.001" ixy="0" ixz="0" iyy="0.001" iyz="0" izz="0.001"/>
+                <mass value="0.006089"/>
+                <inertia ixx="0.000000197597" ixy="-0.000000000005" ixz="0.00000000043" iyy="0.000000404632" iyz="0.000000000054" izz="0.000000440963"/>
             </inertial>
         </link>
@@ -183,6 +183,6 @@
             <inertial>
                 <origin xyz="0 0 0" rpy="0 0 0"/>
-                <mass value="2.0"/>
-                <inertia ixx="0.001" ixy="0" ixz="0" iyy="0.001" iyz="0" izz="0.001"/>
+                <mass value="0.005429"/>
+                <inertia ixx="0.000000155671" ixy="0.000000000024" ixz="0.000000002166" iyy="0.00000033961" iyz="0.000000000002" izz="0.000000357923"/>
             </inertial>
         </link>

File: urdf/macros.xacro (robot description, xacro)
@@ -17,6 +17,6 @@
             <inertial>
                 <origin xyz="0 0 0" rpy="0 0 0"/>
-                <mass value="2.0"/>
-                <inertia ixx="0.01" ixy="0" ixz="0" iyy="0.01" iyz="0" izz="0.01"/>
+                <mass value="0.004836"/>
+                <inertia ixx="0.000000235908" ixy="-0.000000006556" ixz="0.000000001806" iyy="0.000000740439" iyz="0.000000000035" izz="0.000000830731"/>
             </inertial>
         </link>
@@ -57,6 +57,6 @@
             <inertial>
                 <origin xyz="0 0 0" rpy="0 0 0"/>
-                <mass value="2.0"/>
-                <inertia ixx="0.001" ixy="0" ixz="0" iyy="0.001" iyz="0" izz="0.001"/>
+                <mass value="0.001654"/>
+                <inertia ixx="0.000000049479" ixy="0.000000000263" ixz="0.000000000299" iyy="0.000000032432" iyz="0.000000000057" izz="0.000000038462"/>
             </inertial>
         </link>
@@ -98,6 +98,6 @@
             <inertial>
                 <origin xyz="0 0 0" rpy="0 0 0"/>
-                <mass value="2.0"/>
-                <inertia ixx="0.001" ixy="0" ixz="0" iyy="0.001" iyz="0" izz="0.001"/>
+                <mass value="0.005708"/>
+                <inertia ixx="0.00000018835" ixy="0.00000001165" ixz="0.000000000165" iyy="0.000000372084" iyz="-0.000000000039" izz="0.00000039757"/>
             </inertial>
         </link>
@@ -139,6 +139,6 @@
             <inertial>
                 <origin xyz="0 0 0" rpy="0 0 0"/>
-                <mass value="2.0"/>
-                <inertia ixx="0.001" ixy="0" ixz="0" iyy="0.001" iyz="0" izz="0.001"/>
+                <mass value="0.005093"/>
+                <inertia ixx="0.000000143621" ixy="-0.00000000003" ixz="0.000000000091" iyy="0.000000290288" iyz="-0.000000000079" izz="0.000000314107"/>
             </inertial>
         </link>
@@ -180,6 +180,6 @@
             <inertial>
                 <origin xyz="0 0 0" rpy="0 0 0"/>
-                <mass value="2.0"/>
-                <inertia ixx="0.001" ixy="0" ixz="0" iyy="0.001" iyz="0" izz="0.001"/>
+                <mass value="0.005429"/>
+                <inertia ixx="0.000000155634" ixy="0.000000000003" ixz="-0.000000002159" iyy="0.000000339577" iyz="-0.000000000002" izz="0.000000357884"/>
             </inertial>
         </link>

Commit message: update mass of supports

File: urdf/hopejr_hand.urdf (robot description, URDF)
Before this commit: robot hopejr_hand, 46 links, 45 joints
Links:
- link index_dip_1_support: mass 2.0 -> 0.0000000000001
- link index_dip_2_support: mass 2.0 -> 0.0000000000001
- link index_mcp_2_support: mass 2.0 -> 0.0000000000001
- link index_pip_support: mass 2.0 -> 0.0000000000001
- link middle_dip_1_support: mass 2.0 -> 0.0000000000001
- link middle_dip_2_support: mass 2.0 -> 0.0000000000001
- link middle_mcp_2_support: mass 2.0 -> 0.0000000000001
- link middle_pip_support: mass 2.0 -> 0.0000000000001
- link pinky_dip_1_support: mass 2.0 -> 0.0000000000001
- link pinky_dip_2_support: mass 2.0 -> 0.0000000000001
- link pinky_mcp_2_support: mass 2.0 -> 0.0000000000001
- link pinky_pip_support: mass 2.0 -> 0.0000000000001
- link ring_dip_1_support: mass 2.0 -> 0.0000000000001
- link ring_dip_2_support: mass 2.0 -> 0.0000000000001
- link ring_mcp_2_support: mass 2.0 -> 0.0000000000001
- link ring_pip_support: mass 2.0 -> 0.0000000000001
- link thumb_dip_support: mass 2.0 -> 0.0000000000001
- link thumb_pip_1_support: mass 2.0 -> 0.0000000000001
- link thumb_pip_2_support: mass 2.0 -> 0.0000000000001

File: urdf/hopejr_hand.urdf.xacro (robot description, xacro)
@@ -77,6 +77,6 @@
             <inertial>
                 <origin xyz="0 0 0" rpy="0 0 0"/>
-                <mass value="2.0"/>
-                <inertia ixx="0" ixy="0" ixz="0" iyy="0" iyz="0" izz="0"/>
+                <mass value="0.0000000000001"/>
+                <inertia ixx="0.00000000000001" ixy="0" ixz="0" iyy="0.00000000000001" iyz="0" izz="0.00000000000001"/>
             </inertial>
         </link>
@@ -117,6 +117,6 @@
             <inertial>
                 <origin xyz="0 0 0" rpy="0 0 0"/>
-                <mass value="2.0"/>
-                <inertia ixx="0" ixy="0" ixz="0" iyy="0" iyz="0" izz="0"/>
+                <mass value="0.0000000000001"/>
+                <inertia ixx="0.00000000000001" ixy="0" ixz="0" iyy="0.00000000000001" iyz="0" izz="0.00000000000001"/>
             </inertial>
         </link>
@@ -157,6 +157,6 @@
             <inertial>
                 <origin xyz="0 0 0" rpy="0 0 0"/>
-                <mass value="2.0"/>
-                <inertia ixx="0" ixy="0" ixz="0" iyy="0" iyz="0" izz="0"/>
+                <mass value="0.0000000000001"/>
+                <inertia ixx="0.00000000000001" ixy="0" ixz="0" iyy="0.00000000000001" iyz="0" izz="0.00000000000001"/>
             </inertial>
         </link>

File: urdf/macros.xacro (robot description, xacro)
@@ -30,6 +30,6 @@
             <inertial>
                 <origin xyz="0 0 0" rpy="0 0 0"/>
-                <mass value="2.0"/>
-                <inertia ixx="0" ixy="0" ixz="0" iyy="0" iyz="0" izz="0"/>
+                <mass value="0.0000000000001"/>
+                <inertia ixx="0.00000000000001" ixy="0" ixz="0" iyy="0.00000000000001" iyz="0" izz="0.00000000000001"/>
             </inertial>
         </link>
@@ -71,6 +71,6 @@
             <inertial>
                 <origin xyz="0 0 0" rpy="0 0 0"/>
-                <mass value="2.0"/>
-                <inertia ixx="0" ixy="0" ixz="0" iyy="0" iyz="0" izz="0"/>
+                <mass value="0.0000000000001"/>
+                <inertia ixx="0.00000000000001" ixy="0" ixz="0" iyy="0.00000000000001" iyz="0" izz="0.00000000000001"/>
             </inertial>
         </link>
@@ -112,6 +112,6 @@
             <inertial>
                 <origin xyz="0 0 0" rpy="0 0 0"/>
-                <mass value="2.0"/>
-                <inertia ixx="0" ixy="0" ixz="0" iyy="0" iyz="0" izz="0"/>
+                <mass value="0.0000000000001"/>
+                <inertia ixx="0.00000000000001" ixy="0" ixz="0" iyy="0.00000000000001" iyz="0" izz="0.00000000000001"/>
             </inertial>
         </link>
@@ -153,6 +153,6 @@
             <inertial>
                 <origin xyz="0 0 0" rpy="0 0 0"/>
-                <mass value="2.0"/>
-                <inertia ixx="0" ixy="0" ixz="0" iyy="0" iyz="0" izz="0"/>
+                <mass value="0.0000000000001"/>
+                <inertia ixx="0.00000000000001" ixy="0" ixz="0" iyy="0.00000000000001" iyz="0" izz="0.00000000000001"/>
             </inertial>
         </link>
